File: hardware/GSR/GSRv3.0.brd (EAGLE design)
At the start: 67.3 x 52.1 mm, 38 parts, among them U1 ARDUINO_MINI

Commit message: v3.0
Parts:
- removed FET5, FET6: MPSA42, SparkFun-DiscreteSemi:SOT23-3
- removed LED5, LED6: (no value), microbuilder:CHIPLED_0603_NOOUTLINE
- removed R5, R6: 330, SparkFun-Passives:0603-RES
- removed VBAT@1, VBAT@2, W1, W2, W3, W4, W5, W6: (no value), SparkFun-Connectors:1X01NS-KIT
- added WIRE1, WIRE2, WIRE3, WIRE4: (no value), SparkFun-Connectors:1X02
- R7, R8: value 330 -> 1K
- moved R3 12.8 mm to (48.3, 43.8), turned to 180 degrees
- moved LED3 12.7 mm to (48.3, 46.0), turned to 90 degrees
- moved FET3 12.7 mm to (48.3, 38.1), turned to 270 degrees
- moved FET4 8.03 mm to (54.6, 40.6)
- moved R4 7.73 mm to (54.6, 43.8), turned to 180 degrees
- moved LED4 7.68 mm to (54.6, 46.0), turned to 90 degrees
- moved R2 2.84 mm to (34.3, 43.8)
- moved FET2 2.84 mm to (34.3, 38.1)
- moved LED2 2.71 mm to (34.3, 46.0)
- moved R1 1.27 mm to (27.9, 43.8)
- moved LED1 0.95 mm to (27.9, 46.0)
- moved GSR_IN_CAP 0.32 mm to (28.9, 6.35)
Connections:
- removed net FET5: FET5.1, U1.D3
- removed net FET6: FET6.1, U1.D2
- removed net N$5: LED5.C, R5.2
- removed net N$6: LED6.C, R6.2
- removed net WIRE5: FET5.3, R5.1, W5.1
- removed net WIRE6: FET6.3, R6.1, W6.1
- net DEBUG_VCC: no longer LED5.A, LED6.A
- net FET1: now also U1.D5; no longer U1.D9
- net FET2: now also U1.D4; no longer U1.D8
- net FET3: now also U1.D3; no longer U1.D5
- net FET4: now also U1.D2; no longer U1.D4
- net GND: no longer FET5.2, FET6.2
- net GSR_SIG: now also U1.A5; no longer U1.A7
- net VBAT: now also WIRE1.1, WIRE2.1, WIRE3.1, WIRE4.1; no longer VBAT@1.1, VBAT@2.1
- net WIRE1: now also WIRE1.2; no longer W1.1
- net WIRE2: now also WIRE2.2; no longer W2.1
- net WIRE3: now also WIRE3.2; no longer W3.1
- net WIRE4: now also WIRE4.2; no longer W4.1
Routing:
- net WIRE5: track 25.9 -> 0.00 mm
- net WIRE6: track 22.8 -> 0.00 mm
- net FET6: track 12.5 -> 0.00 mm, vias 1 -> 0
- net FET5: track 11.4 -> 0.00 mm, vias 1 -> 0
- net WIRE4: track 29.3 -> 19.7 mm
- net FET1: track 6.94 -> 14.1 mm, vias 1 -> 2
- net GND: track 25.1 -> 18.5 mm, vias 5 -> 6
- net FET4: track 8.43 -> 14.3 mm, vias 0 -> 2
- net WIRE3: track 28.2 -> 24.8 mm
- net FET3: track 4.13 -> 7.03 mm
- net GSR_VCC: track 15.8 -> 13.0 mm
- net WIRE1: track 22.0 -> 19.7 mm
- net N$6: track 1.95 -> 0.00 mm, vias 0 -> 1
- net N$5: track 1.95 -> 0.00 mm
- net GSR_SIG: track 16.7 -> 15.6 mm
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- added copper zone on layer 16, net GND
Other:
- board size 67.3 x 52.1 mm -> 66.2 x 52.1 mm
