File: hardware/GSR/GSRv3.0.sch (EAGLE design)
At the start: 38 parts, among them U1 ARDUINO_MINI

Commit message: v3.0
Parts:
- removed C2, C4: (no value), microbuilder:CAP_CERAMIC0603
- removed FET5, FET6: MPSA42, SparkFun-DiscreteSemi:TRANSISTOR_NPNMPSA42
- removed LED5, LED6: (no value), microbuilder:LED0603_NOOUTLINE
- removed R5, R6: 330, SparkFun-Passives:RESISTOR0603-RES
- removed VBAT@1, VBAT@2, W1, W2, W3, W4, W5, W6: (no value), SparkFun-Connectors:M01NOSILK-KIT
- added GSR_IN_CAP, GSR_OUT_CAP: 1uF, microbuilder:CAP_CERAMIC0603
- added WIRE1, WIRE2, WIRE3, WIRE4: (no value), SparkFun-Connectors:M02PTH
- R7, R8: value 330 -> 1K
Connections:
- removed net FET5: FET5.B, U1.D3
- removed net FET6: FET6.B, U1.D2
- removed net N$5: LED5.C, R5.2
- removed net N$6: LED6.C, R6.2
- removed net N$7: POWER.2
- removed net WIRE5: FET5.C, R5.1, W5.1
- removed net WIRE6: FET6.C, R6.1, W6.1
- net DEBUG_VCC: no longer LED5.A, LED6.A
- net FET1: now also U1.D5; no longer U1.D9
- net FET2: now also U1.D4; no longer U1.D8
- net FET3: now also U1.D3; no longer U1.D5
- net FET4: now also U1.D2; no longer U1.D4
- net GND: now also GSR_IN_CAP.P$1, GSR_OUT_CAP.P$1, POWER.2; no longer FET5.E, FET6.E
- net GSR_SIG: now also U1.A5; no longer U1.A7
- net GSR_VCC: now also GSR_OUT_CAP.P$2
- net VBAT: now also GSR_IN_CAP.P$2, WIRE1.1, WIRE2.1, WIRE3.1, WIRE4.1; no longer VBAT@1.1, VBAT@2.1
- net WIRE1: now also WIRE1.2; no longer W1.1
- net WIRE2: now also WIRE2.2; no longer W2.1
- net WIRE3: now also WIRE3.2; no longer W3.1
- net WIRE4: now also WIRE4.2; no longer W4.1
Other:
- moved on the sheet: FET1, FET2, FET3, FET4, GSR, LED1, LED2, LED3, LED4, R1, R2, R3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
