File: hardware/GSR/GSRv3.1.sch (EAGLE design)
At the start: 28 parts, among them U1 ARDUINO_MINI

Commit message: GSR3.2
Parts:
- removed GSR: (no value), SparkFun-Connectors:M04PTH
- added JP1: (no value), SparkFun-Connectors:M04POLAR
- added JP2: (no value), SparkFun-Connectors:M06SILK_FEMALE_PTH
- added R10, R5, R6, R9: 1K, microbuilder:RESISTOR0603
- WIRE1, WIRE2, WIRE3, WIRE4: device SparkFun-Connectors:M02PTH -> SparkFun-Connectors:M02POLAR
Connections:
- removed net AIN0: U1.D6
- removed net AIN1: U1.D7
- new net A0: JP2.1, U1.A5
- new net A1: JP2.2, U1.A4
- new net D0: JP2.3, U1.D9
- new net D1: JP2.4, U1.D8
- new net D2: JP2.5, U1.D7
- new net D3: JP2.6, U1.D6
- new net N$5: FET1.B, R5.2
- new net N$6: FET2.B, R6.1
- new net N$7: FET3.B, R9.2
- new net N$8: FET4.B, R10.2
- net FET1: now also R5.1; no longer FET1.B
- net FET2: now also R6.2; no longer FET2.B
- net FET3: now also R9.1; no longer FET3.B
- net FET4: now also R10.1; no longer FET4.B
- net GND: now also JP1.3; no longer GSR.2
- net GSR_SIG: now also JP1.1, U1.A7; no longer GSR.4, U1.A5
- net GSR_VCC: now also JP1.4; no longer GSR.1
- net GSR_VSS: now also JP1.2; no longer GSR.3
Other:
- moved on the sheet: FET1, FET2, FET3, FET4, WIRE1, WIRE2, WIRE3, WIRE4
