File: hardware/GSR/GSRv3.2.brd (EAGLE design)
At the start: 66.3 x 52.1 mm, 32 parts, among them U1 ARDUINO_MINI

Commit message: GSR3.2
Parts:
- added JP2: (no value), SparkFun-Connectors:1X06
- moved WIRE4 3.59 mm to (70.5, 31.1)
- moved WIRE2 3.59 mm to (15.2, 27.9)
- moved WIRE1 3.59 mm to (10.2, 33.0)
- moved WIRE3 3.59 mm to (65.4, 26.0)
Connections:
- removed net AIN0: U1.D6
- removed net AIN1: U1.D7
- new net A0: JP2.1, U1.A5
- new net A1: JP2.2, U1.A4
- new net D0: JP2.3, U1.D9
- new net D1: JP2.4, U1.D8
- new net D2: JP2.5, U1.D7
- new net D3: JP2.6, U1.D6
- net GSR_SIG: now also U1.A7; no longer U1.A5
Routing:
- net D3: track 0.00 -> 18.2 mm
- net A0: track 0.00 -> 18.0 mm
- net D2: track 0.00 -> 17.3 mm
- net A1: track 0.00 -> 15.9 mm
- net D1: track 0.00 -> 15.2 mm
- net D0: track 0.00 -> 13.8 mm
- net WIRE1: track 18.7 -> 22.3 mm
- net WIRE2: track 25.1 -> 28.7 mm
- net WIRE3: track 25.4 -> 29.0 mm
- net WIRE4: track 19.0 -> 22.6 mm
- net GSR_SIG: track 16.2 -> 19.3 mm
- net FET1: track 11.9 -> 10.3 mm
- net FET4: track 11.9 -> 10.3 mm
- net GSR_VCC: track 16.5 -> 17.6 mm
- net GND: vias 7 -> 8
Other:
- board size 66.3 x 52.1 mm -> 71.3 x 50.8 mm
- board text added: "revC"
- board text added: "smarTee"
